File: Amiga-MouseTrigger.kicad_sch (KiCad schematic)
At the start: 11 parts, among them J1 INPUT_SIGNALS, J2 OUTPUT, J3 POWER, J99 OSHW_LOGO, U1 74LS74

Commit message: Replace THT elements with SMD.
Other:
- company: SukkoPera -> k0lo
- title: OpenAmigaMouseTrigger -> Amiga-MouseTrigger
Changed lines of the file:
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@@
   (paper "A4")
   (title_block
-    (title "OpenAmigaMouseTrigger")
-    (date "2018-05-29")
-    (rev "2")
-    (company "SukkoPera")
+    (title "Amiga-MouseTrigger")
+    (date "2024-12-30")
+    (rev "3")
+    (company "k0lo")
   )
   (junction (at 132.08 104.14) (diameter 0) (color 0 0 0 0)
@@
     (pin "1")
     (instances
-      (project "OpenAmigaMouseTrigger"
+      (project "Amiga-MouseTrigger"
         (path "/2dc521a5-7c7d-4b09-a132-5a2b0ad5558e"
           (reference "J1") (unit 1)
@@
     (pin "2")
     (instances
-      (project "OpenAmigaMouseTrigger"
+      (project "Amiga-MouseTrigger"
         (path "/2dc521a5-7c7d-4b09-a132-5a2b0ad5558e"
           (reference "C1") (unit 1)
@@
     (pin "2")
     (instances
-      (project "OpenAmigaMouseTrigger"
+      (project "Amiga-MouseTrigger"
         (path "/2dc521a5-7c7d-4b09-a132-5a2b0ad5558e"
           (reference "R3") (unit 1)
@@
     (pin "14")
     (instances
-      (project "OpenAmigaMouseTrigger"
+      (project "Amiga-MouseTrigger"
         (path "/2dc521a5-7c7d-4b09-a132-5a2b0ad5558e"
           (reference "U1") (unit 1)
@@
     (pin "9")
     (instances
-      (project "OpenAmigaMouseTrigger"
+      (project "Amiga-MouseTrigger"
         (path "/2dc521a5-7c7d-4b09-a132-5a2b0ad5558e"
           (reference "U1") (unit 2)
@@
     (pin "1")
     (instances
-      (project "OpenAmigaMouseTrigger"
+      (project "Amiga-MouseTrigger"
         (path "/2dc521a5-7c7d-4b09-a132-5a2b0ad5558e"
           (reference "#PWR01") (unit 1)
@@
     (pin "1")
     (instances
-      (project "OpenAmigaMouseTrigger"
+      (project "Amiga-MouseTrigger"
         (path "/2dc521a5-7c7d-4b09-a132-5a2b0ad5558e"
           (reference "#PWR02") (unit 1)
@@
     (pin "2")
     (instances
-      (project "OpenAmigaMouseTrigger"
+      (project "Amiga-MouseTrigger"
         (path "/2dc521a5-7c7d-4b09-a132-5a2b0ad5558e"
           (reference "J2") (unit 1)
@@
     (pin "2")
     (instances
-      (project "OpenAmigaMouseTrigger"
+      (project "Amiga-MouseTrigger"
         (path "/2dc521a5-7c7d-4b09-a132-5a2b0ad5558e"
           (reference "C2") (unit 1)
@@
     (pin "1")
     (instances
-      (project "OpenAmigaMouseTrigger"
+      (project "Amiga-MouseTrigger"
         (path "/2dc521a5-7c7d-4b09-a132-5a2b0ad5558e"
           (reference "#PWR03") (unit 1)
@@
     (pin "1")
     (instances
-      (project "OpenAmigaMouseTrigger"
+      (project "Amiga-MouseTrigger"
         (path "/2dc521a5-7c7d-4b09-a132-5a2b0ad5558e"
           (reference "#PWR04") (unit 1)
@@
     (pin "1")
     (instances
-      (project "OpenAmigaMouseTrigger"
+      (project "Amiga-MouseTrigger"
         (path "/2dc521a5-7c7d-4b09-a132-5a2b0ad5558e"
           (reference "#PWR05") (unit 1)
@@
     (pin "1")
     (instances
-      (project "OpenAmigaMouseTrigger"
+      (project "Amiga-MouseTrigger"
         (path "/2dc521a5-7c7d-4b09-a132-5a2b0ad5558e"
           (reference "#PWR06") (unit 1)
@@
     (pin "1")
     (instances
-      (project "OpenAmigaMouseTrigger"
+      (project "Amiga-MouseTrigger"
         (path "/2dc521a5-7c7d-4b09-a132-5a2b0ad5558e"
           (reference "#FLG07") (unit 1)
@@
     (pin "1")
     (instances
-      (project "OpenAmigaMouseTrigger"
+      (project "Amiga-MouseTrigger"
         (path "/2dc521a5-7c7d-4b09-a132-5a2b0ad5558e"
           (reference "#FLG08") (unit 1)
@@
     (pin "2")
     (instances
-      (project "OpenAmigaMouseTrigger"
+      (project "Amiga-MouseTrigger"
         (path "/2dc521a5-7c7d-4b09-a132-5a2b0ad5558e"
           (reference "J3") (unit 1)
@@
     (pin "1")
     (instances
-      (project "OpenAmigaMouseTrigger"
+      (project "Amiga-MouseTrigger"
         (path "/2dc521a5-7c7d-4b09-a132-5a2b0ad5558e"
           (reference "#PWR09") (unit 1)
@@
     (pin "1")
     (instances
-      (project "OpenAmigaMouseTrigger"
+      (project "Amiga-MouseTrigger"
         (path "/2dc521a5-7c7d-4b09-a132-5a2b0ad5558e"
           (reference "#PWR010") (unit 1)
@@
     (pin "1")
     (instances
-      (project "OpenAmigaMouseTrigger"
+      (project "Amiga-MouseTrigger"
         (path "/2dc521a5-7c7d-4b09-a132-5a2b0ad5558e"
           (reference "#PWR011") (unit 1)
@@
     (pin "1")
     (instances
-      (project "OpenAmigaMouseTrigger"
+      (project "Amiga-MouseTrigger"
         (path "/2dc521a5-7c7d-4b09-a132-5a2b0ad5558e"
           (reference "J99") (unit 1)
@@
     (pin "2")
     (instances
-      (project "OpenAmigaMouseTrigger"
+      (project "Amiga-MouseTrigger"
         (path "/2dc521a5-7c7d-4b09-a132-5a2b0ad5558e"
           (reference "R1") (unit 1)
@@
     (pin "2")
     (instances
-      (project "OpenAmigaMouseTrigger"
+      (project "Amiga-MouseTrigger"
         (path "/2dc521a5-7c7d-4b09-a132-5a2b0ad5558e"
           (reference "R2") (unit 1)
@@
     (pin "2")
     (instances
-      (project "OpenAmigaMouseTrigger"
+      (project "Amiga-MouseTrigger"
         (path "/2dc521a5-7c7d-4b09-a132-5a2b0ad5558e"
           (reference "R4") (unit 1)
